Commit message: urdf_camera_table_add

File: panda_description/urdf/panda.urdf (robot description, URDF)
Before this commit: robot panda, 12 links, 11 joints
Links:
- added link static_camera; visual mesh filename=package://moveit_resources_panda_description/meshes/visual/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
- added link table; visual box size=1.0 1.0 0.3
Joints:
- added joint base_to_static_camera: type fixed, parent panda_link0, child static_camera, origin xyz=1.0 0 1.0 rpy=0 3.14 0, axis 0 0 0
- added joint panda_link0_to_table: type fixed, parent panda_link0, child table, origin xyz=0 0 0 rpy=0 0 0, axis 0 0 0

Commit message: Revert "urdf_camera_table_add"
This reverts commit b0930ba109060ea70396dd405a9875ee84a10278.

File: panda_description/urdf/panda.urdf (robot description, URDF)
Before this commit: robot panda, 14 links, 13 joints
Links:
- removed link static_camera
- removed link table
Joints:
- removed joint base_to_static_camera
- removed joint panda_link0_to_table
